Commit message: Initial commit: HomeCleanerBot - Autonomous Indoor Cleaning Robot with ROS2 and Gazebo

File: src/auto_robot/description/robot_core.xacro (robot description, xacro)
@@ -20,8 +20,8 @@
     </material>
     <material name="orange">
-        <color rgba="1 0.3 0.1 1"/>
+        <color rgba="1 0.6 0.2 1"/>
     </material>
     <material name="blue">
-        <color rgba="0.2 0.2 1 1"/>
+        <color rgba="0.2 0.6 1 1"/>
     </material>
     <material name="black">
@@ -29,8 +29,11 @@
     </material>
     <material name="red">
-        <color rgba="1 0 0 1"/>
+        <color rgba="0.8 0.1 0.1 1"/>
     </material>
     <material name="green">
-        <color rgba="0 1 0 1"/>
+        <color rgba="0.2 0.8 0.2 1"/>
+    </material>
+    <material name="silver">
+        <color rgba="0.75 0.75 0.75 1"/>
     </material>
     <!-- BASE LINK -->
@@ -59,4 +62,11 @@
             <material name="red"/>
         </visual>
+        <visual>
+            <origin xyz="${chassis_length/1.5} 0 ${chassis_height/1.2}"/>
+            <geometry>
+                <box size="${chassis_length/3} ${chassis_width/1.5} ${chassis_height/2}"/>
+            </geometry>
+            <material name="white"/>
+        </visual>
         <collision>
             <origin xyz="${chassis_length/2} 0 ${chassis_height/2}"/>
@@ -81,8 +91,16 @@
     <link name="left_wheel">
         <visual>
+            <origin xyz="0 0 0" rpy="0 0 0"/>
             <geometry>
                 <cylinder radius="${wheel_radius}" length="${wheel_thickness}"/>
             </geometry>
             <material name="green"/>
+        </visual>
+        <visual>
+            <origin xyz="0 0 0" rpy="0 0 0"/>
+            <geometry>
+                <cylinder radius="${wheel_radius/1.5}" length="${wheel_thickness/1.2}"/>
+            </geometry>
+            <material name="black"/>
         </visual>
         <collision>
@@ -107,8 +125,16 @@
     <link name="right_wheel">
         <visual>
+            <origin xyz="0 0 0" rpy="0 0 0"/>
             <geometry>
                 <cylinder radius="${wheel_radius}" length="${wheel_thickness}"/>
             </geometry>
             <material name="green"/>
+        </visual>
+        <visual>
+            <origin xyz="0 0 0" rpy="0 0 0"/>
+            <geometry>
+                <cylinder radius="${wheel_radius/1.5}" length="${wheel_thickness/1.2}"/>
+            </geometry>
+            <material name="black"/>
         </visual>
         <collision>
@@ -132,8 +158,16 @@
     <link name="caster_wheel">
         <visual>
+            <origin xyz="0 0 0" rpy="0 0 0"/>
             <geometry>
                 <sphere radius="${caster_wheel_radius}"/>
             </geometry>
             <material name="black"/>
+        </visual>
+        <visual>
+            <origin xyz="0 0 0" rpy="0 0 0"/>
+            <geometry>
+                <sphere radius="${caster_wheel_radius/2}"/>
+            </geometry>
+            <material name="silver"/>
         </visual>
         <collision>
